Commit message: 

File: urdf/aros.urdf (robot description, URDF)
Before this commit: robot aros, 8 links, 7 joints
Links:
- added link right_adapter_link; visual mesh filename=package://aros_description/meshes/right_arm/adapter/body.dae
- added link right_arm3_link; visual mesh filename=package://aros_description/meshes/right_arm/link3/body.dae
- added link right_arm4_link; visual mesh filename=package://aros_description/meshes/right_arm/link4/body.dae
- added link right_arm5_link; visual mesh filename=package://aros_description/meshes/right_arm/link5/body.dae
- added link right_arm6_link; visual mesh filename=package://aros_description/meshes/right_arm/link6/body.dae
- added link right_arm7_link; visual mesh filename=package://aros_description/meshes/right_arm/link7/body.dae
- added link right_finger3_1_link; visual mesh filename=package://aros_description/meshes/right_arm/fingers/finger3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
- added link right_finger3_2_link; visual mesh filename=package://aros_description/meshes/right_arm/fingers/finger3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
- added link right_finger3_tip_link; visual mesh filename=package://aros_description/meshes/right_arm/fingers/finger3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
- added link right_fts_link; visual mesh filename=package://aros_description/meshes/right_arm/fts/body.dae
- added link right_hand_link; visual mesh filename=package://aros_description/meshes/right_arm/barrett_hand/bo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
- added link right_hand_sensor_link; visual mesh filename=package://aros_description/meshes/right_arm/hand_sensor/bod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
Joints:
- added joint right_finger3_joint1: type revolute, parent right_hand_link, child right_finger3_1_link, origin xyz=0.03 0 -0.05 rpy=1.57 3.14 0, axis 0 0 1, limit lower=0 upper=2.44 effort=160.0 velocity=0.5
- added joint right_finger3_joint2: type revolute, parent right_finger3_1_link, child right_finger3_2_link, origin xyz=-0.005 0.07 0 rpy=0 0 0, axis 0 0 1, limit lower=0 upper=0.79 effort=160.0 velocity=0.5
- added joint right_fixed_joint1: type fixed, parent right_arm7_link, child right_fts_link, origin xyz=0 0 0.065 rpy=-1.57 -1.57 0
- added joint right_fixed_joint2: type fixed, parent right_fts_link, child right_adapter_link, origin xyz=0.04 0 0 rpy=0 0 0
- added joint right_fixed_joint3: type fixed, parent right_adapter_link, child right_hand_link, origin xyz=0.06 0 0 rpy=0 0 0
- added joint right_fixed_joint4: type fixed, parent right_hand_link, child right_hand_sensor_link, origin xyz=0.035 0 0 rpy=0 0 0
- added joint right_fixed_joint5: type fixed, parent right_finger3_2_link, child right_finger3_tip_link, origin xyz=-0.028 0.022 0 rpy=0 0 1.97
- added joint right_joint2: type revolute, parent right_arm2_link, child right_arm3_link, origin xyz=-0.195 0 0 rpy=-1.57 0 1.57, axis 0 0 1, limit lower=-1.57 upper=2.44 effort=160.0 velocity=0.5
- added joint right_joint3: type revolute, parent right_arm3_link, child right_arm4_link, origin xyz=0 0 0.2 rpy=1.57 1.57 0, axis 0 0 1, limit lower=-2.88 upper=0.26 effort=160.0 velocity=0.5
- added joint right_joint4: type revolute, parent right_arm4_link, child right_arm5_link, origin xyz=-0.208 0 0 rpy=-1.57 0 1.57, axis 0 0 1, limit lower=-2.88 upper=2.88 effort=160.0 velocity=0.5
- added joint right_joint5: type revolute, parent right_arm5_link, child right_arm6_link, origin xyz=0 0 0.161 rpy=1.57 1.57 0, axis 0 0 1, limit lower=-2.09 upper=2.09 effort=160.0 velocity=0.5
- added joint right_joint6: type revolute, parent right_arm6_link, child right_arm7_link, origin xyz=-0.053 0 0 rpy=-1.57 0 1.57, axis 0 0 1, limit lower=-1.57 upper=2.88 effort=160.0 velocity=0.5

Commit message: 

File: urdf/aros.urdf (robot description, URDF)
Before this commit: robot aros, 20 links, 19 joints
Links:
- added link right_finger1_base_link; visual mesh filename=package://aros_description/meshes/right_arm/fingers/finger1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
Joints:
- added joint right_finger1_base_joint: type revolute, parent right_hand_link, child right_finger1_base_link, origin xyz=0 -0.025 0 rpy=0 1.57 0, axis 0 0 1, limit lower=0 upper=3.14 effort=160.0 velocity=0.5

Commit message: 

File: urdf/aros.urdf (robot description, URDF)
Before this commit: robot aros, 21 links, 20 joints
Links:
- added link right_finger2_base_link; visual mesh filename=package://aros_description/meshes/right_arm/fingers/finger2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
- link base_link: geometry collision mesh filename=package://aros_description/meshes/base/link.dae; visual mesh filename=package://aros_description/meshes/base/body.dae
- link right_arm0_link: geometry collision mesh filename=package://aros_description/meshes/right_arm/link0/link.dae; visual mesh filename=package://aros_description/meshes/right_arm/link0/body.dae
- link right_arm1_link: geometry collision mesh filename=package://aros_description/meshes/right_arm/link1/link.dae; visual mesh filename=package://aros_description/meshes/right_arm/link1/body.dae
- link right_arm2_link: geometry collision mesh filename=package://aros_description/meshes/right_arm/link2/link.dae; visual mesh filename=package://aros_description/meshes/right_arm/link2/body.dae
- link right_arm3_link: geometry collision mesh filename=package://aros_description/meshes/right_arm/link3/link.dae; visual mesh filename=package://aros_description/meshes/right_arm/link3/body.dae
Joints:
- added joint right_finger2_base_joint: type revolute, parent right_hand_link, child right_finger2_base_link, origin xyz=0 0.025 0 rpy=0 1.57 0, axis 0 0 1, limit lower=-3.14 upper=0 effort=160.0 velocity=0.5

Commit message: added some links

File: urdf/aros.urdf (robot description, URDF)
Before this commit: robot aros, 22 links, 21 joints
Links:
- link right_arm4_link: geometry collision mesh filename=package://aros_description/meshes/right_arm/link4/link.dae; visual mesh filename=package://aros_description/meshes/right_arm/link4/body.dae
- link right_arm5_link: geometry collision mesh filename=package://aros_description/meshes/right_arm/link5/link.dae; visual mesh filename=package://aros_description/meshes/right_arm/link5/body.dae
- link right_arm6_link: geometry collision mesh filename=package://aros_description/meshes/right_arm/link6/link.dae; visual mesh filename=package://aros_description/meshes/right_arm/link6/body.dae
- link right_arm7_link: geometry collision mesh filename=package://aros_description/meshes/right_arm/link7/link.dae; visual mesh filename=package://aros_description/meshes/right_arm/link7/body.dae
- link right_finger1_base_link: geometry collision mesh filename=package://aros_description/meshes/right_arm/fingers/finger1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; visual mesh filename=package://aros_description/meshes/right_arm/fingers/finger1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
- link right_finger2_base_link: geometry collision mesh filename=package://aros_description/meshes/right_arm/fingers/finger2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; visual mesh filename=package://aros_description/meshes/right_arm/fingers/finger2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
- link right_finger3_1_link: geometry collision mesh filename=package://aros_description/meshes/right_arm/fingers/finger3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; visual mesh filename=package://aros_description/meshes/right_arm/fingers/finger3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
- link right_finger3_2_link: geometry collision mesh filename=package://aros_description/meshes/right_arm/fingers/finger3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; visual mesh filename=package://aros_description/meshes/right_arm/fingers/finger3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
- link right_fts_link: geometry collision mesh filename=package://aros_description/meshes/right_arm/fts/link.dae; visual mesh filename=package://aros_description/meshes/right_arm/fts/body.dae
- link right_hand_link: geometry collision mesh filename=package://aros_description/meshes/right_arm/barrett_hand/li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; visual mesh filename=package://aros_description/meshes/right_arm/barrett_hand/bo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

Commit message: 

File: urdf/aros.urdf (robot description, URDF)
Before this commit: robot aros, 22 links, 21 joints
Links:
- added link right_finger1_1_link; collision mesh filename=package://aros_description/meshes/right_arm/fingers/finger1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; visual mesh filename=package://aros_description/meshes/right_arm/fingers/finger1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
- added link right_finger1_2_link; collision mesh filename=package://aros_description/meshes/right_arm/fingers/finger1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; visual mesh filename=package://aros_description/meshes/right_arm/fingers/finger1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
Joints:
- added joint right_finger1_joint1: type revolute, parent right_finger1_base_link, child right_finger1_1_link, origin xyz=-0.05 0 0.036 rpy=0 1.57 1.57, axis 0 0 1, limit lower=0 upper=2.44 effort=160.0 velocity=0.5
- added joint right_finger1_joint2: type revolute, parent right_finger1_1_link, child right_finger1_2_link, origin xyz=-0.005 0.07 0 rpy=0 0 0, axis 0 0 1, limit lower=0 upper=0.79 effort=160.0 velocity=0.5

Commit message: right arm completed

File: urdf/aros.urdf (robot description, URDF)
Before this commit: robot aros, 24 links, 23 joints
Links:
- added link right_finger1_tip_link; visual mesh filename=package://aros_description/meshes/hand/fingers/finger1/tip/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
- added link right_finger2_1_link; collision mesh filename=package://aros_description/meshes/hand/fingers/finger2/link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; visual mesh filename=package://aros_description/meshes/hand/fingers/finger2/link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
- added link right_finger2_2_link; collision mesh filename=package://aros_description/meshes/hand/fingers/finger2/link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; visual mesh filename=package://aros_description/meshes/hand/fingers/finger2/link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
- added link right_finger2_tip_link; visual mesh filename=package://aros_description/meshes/hand/fingers/finger2/tip/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
- link right_adapter_link: geometry visual mesh filename=package://aros_description/meshes/hand/adapter/body.dae
- link right_arm0_link: geometry collision mesh filename=package://aros_description/meshes/arm/link0/link.dae; visual mesh filename=package://aros_description/meshes/arm/link0/body.dae
- link right_arm1_link: geometry collision mesh filename=package://aros_description/meshes/arm/link1/link.dae; visual mesh filename=package://aros_description/meshes/arm/link1/body.dae
- link right_arm2_link: geometry collision mesh filename=package://aros_description/meshes/arm/link2/link.dae; visual mesh filename=package://aros_description/meshes/arm/link2/body.dae
- link right_arm3_link: geometry collision mesh filename=package://aros_description/meshes/arm/link3/link.dae; visual mesh filename=package://aros_description/meshes/arm/link3/body.dae
- link right_arm4_link: geometry collision mesh filename=package://aros_description/meshes/arm/link4/link.dae; visual mesh filename=package://aros_description/meshes/arm/link4/body.dae
- link right_arm5_link: geometry collision mesh filename=package://aros_description/meshes/arm/link5/link.dae; visual mesh filename=package://aros_description/meshes/arm/link5/body.dae
- link right_arm6_link: geometry collision mesh filename=package://aros_description/meshes/arm/link6/link.dae; visual mesh filename=package://aros_description/meshes/arm/link6/body.dae
- link right_arm7_link: geometry collision mesh filename=package://aros_description/meshes/arm/link7/link.dae; visual mesh filename=package://aros_description/meshes/arm/link7/body.dae
- link right_finger1_1_link: geometry collision mesh filename=package://aros_description/meshes/hand/fingers/finger1/link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; visual mesh filename=package://aros_description/meshes/hand/fingers/finger1/link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
- link right_finger1_2_link: geometry collision mesh filename=package://aros_description/meshes/hand/fingers/finger1/link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; visual mesh filename=package://aros_description/meshes/hand/fingers/finger1/link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
- link right_finger1_base_link: geometry collision mesh filename=package://aros_description/meshes/hand/fingers/finger1/base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; visual mesh filename=package://aros_description/meshes/hand/fingers/finger1/base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
- link right_finger2_base_link: geometry collision mesh filename=package://aros_description/meshes/hand/fingers/finger2/base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; visual mesh filename=package://aros_description/meshes/hand/fingers/finger2/base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
- link right_finger3_1_link: geometry collision mesh filename=package://aros_description/meshes/hand/fingers/finger3/link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; visual mesh filename=package://aros_description/meshes/hand/fingers/finger3/link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
- link right_finger3_2_link: geometry collision mesh filename=package://aros_description/meshes/hand/fingers/finger3/link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; visual mesh filename=package://aros_description/meshes/hand/fingers/finger3/link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
- link right_finger3_tip_link: geometry visual mesh filename=package://aros_description/meshes/hand/fingers/finger3/tip/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
- link right_fts_link: geometry collision mesh filename=package://aros_description/meshes/hand/fts/link.dae; visual mesh filename=package://aros_description/meshes/hand/fts/body.dae
- link right_hand_link: geometry collision mesh filename=package://aros_description/meshes/hand/barrett_hand/link.dae; visual mesh filename=package://aros_description/meshes/hand/barrett_hand/body.dae
- link right_hand_sensor_link: geometry visual mesh filename=package://aros_description/meshes/hand/hand_sensor/body.dae
Joints:
- added joint right_finger2_joint1: type revolute, parent right_finger2_base_link, child right_finger2_1_link, origin xyz=-0.05 0 0.036 rpy=0 1.57 1.57, axis 0 0 1, limit lower=0 upper=2.44 effort=160.0 velocity=0.5
- added joint right_finger2_joint2: type revolute, parent right_finger2_1_link, child right_finger2_2_link, origin xyz=-0.005 0.07 0 rpy=0 0 0, axis 0 0 1, limit lower=0 upper=0.79 effort=160.0 velocity=0.5
- added joint right_fixed_joint6: type fixed, parent right_finger1_2_link, child right_finger1_tip_link, origin xyz=-0.028 0.022 0 rpy=0 0 1.97
- added joint right_fixed_joint7: type fixed, parent right_finger2_2_link, child right_finger2_tip_link, origin xyz=-0.028 0.022 0 rpy=0 0 1.97

Commit message: first version of the urdf has been completed

File: urdf/aros.urdf (robot description, URDF)
Before this commit: robot aros, 28 links, 27 joints
Links:
- added link left_adapter_link; visual mesh filename=package://aros_description/meshes/hand/adapter/body.dae
- added link left_arm0_link; collision mesh filename=package://aros_description/meshes/arm/link0/link.dae; visual mesh filename=package://aros_description/meshes/arm/link0/body.dae
- added link left_arm1_link; collision mesh filename=package://aros_description/meshes/arm/link1/link.dae; visual mesh filename=package://aros_description/meshes/arm/link1/body.dae
- added link left_arm2_link; collision mesh filename=package://aros_description/meshes/arm/link2/link.dae; visual mesh filename=package://aros_description/meshes/arm/link2/body.dae
- added link left_arm3_link; collision mesh filename=package://aros_description/meshes/arm/link3/link.dae; visual mesh filename=package://aros_description/meshes/arm/link3/body.dae
- added link left_arm4_link; collision mesh filename=package://aros_description/meshes/arm/link4/link.dae; visual mesh filename=package://aros_description/meshes/arm/link4/body.dae
- added link left_arm5_link; collision mesh filename=package://aros_description/meshes/arm/link5/link.dae; visual mesh filename=package://aros_description/meshes/arm/link5/body.dae
- added link left_arm6_link; collision mesh filename=package://aros_description/meshes/arm/link6/link.dae; visual mesh filename=package://aros_description/meshes/arm/link6/body.dae
- added link left_arm7_link; collision mesh filename=package://aros_description/meshes/arm/link7/link.dae; visual mesh filename=package://aros_description/meshes/arm/link7/body.dae
- added link left_finger1_1_link; collision mesh filename=package://aros_description/meshes/hand/fingers/finger1/link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; visual mesh filename=package://aros_description/meshes/hand/fingers/finger1/link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
- added link left_finger1_2_link; collision mesh filename=package://aros_description/meshes/hand/fingers/finger1/link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; visual mesh filename=package://aros_description/meshes/hand/fingers/finger1/link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
- added link left_finger1_base_link; collision mesh filename=package://aros_description/meshes/hand/fingers/finger1/base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; visual mesh filename=package://aros_description/meshes/hand/fingers/finger1/base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
- added link left_finger1_tip_link; visual mesh filename=package://aros_description/meshes/hand/fingers/finger1/tip/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
- added link left_finger2_1_link; collision mesh filename=package://aros_description/meshes/hand/fingers/finger2/link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; visual mesh filename=package://aros_description/meshes/hand/fingers/finger2/link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
- added link left_finger2_2_link; collision mesh filename=package://aros_description/meshes/hand/fingers/finger2/link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; visual mesh filename=package://aros_description/meshes/hand/fingers/finger2/link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
- added link left_finger2_base_link; collision mesh filename=package://aros_description/meshes/hand/fingers/finger2/base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; visual mesh filename=package://aros_description/meshes/hand/fingers/finger2/base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
- added link left_finger2_tip_link; visual mesh filename=package://aros_description/meshes/hand/fingers/finger2/tip/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
- added link left_finger3_1_link; collision mesh filename=package://aros_description/meshes/hand/fingers/finger3/link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; visual mesh filename=package://aros_description/meshes/hand/fingers/finger3/link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
- added link left_finger3_2_link; collision mesh filename=package://aros_description/meshes/hand/fingers/finger3/link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; visual mesh filename=package://aros_description/meshes/hand/fingers/finger3/link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
- added link left_finger3_tip_link; visual mesh filename=package://aros_description/meshes/hand/fingers/finger3/tip/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
- added link left_fts_link; collision mesh filename=package://aros_description/meshes/hand/fts/link.dae; visual mesh filename=package://aros_description/meshes/hand/fts/body.dae
- added link left_hand_link; collision mesh filename=package://aros_description/meshes/hand/barrett_hand/link.dae; visual mesh filename=package://aros_description/meshes/hand/barrett_hand/body.dae
- added link left_hand_sensor_link; visual mesh filename=package://aros_description/meshes/hand/hand_sensor/body.dae
Joints:
- added joint left_finger1_base_joint: type revolute, parent left_hand_link, child left_finger1_base_link, origin xyz=0 -0.025 0 rpy=0 1.57 0, axis 0 0 1, limit lower=0 upper=3.14 effort=160.0 velocity=0.5
- added joint left_finger1_joint1: type revolute, parent left_finger1_base_link, child left_finger1_1_link, origin xyz=-0.05 0 0.036 rpy=0 1.57 1.57, axis 0 0 1, limit lower=0 upper=2.44 effort=160.0 velocity=0.5
- added joint left_finger1_joint2: type revolute, parent left_finger1_1_link, child left_finger1_2_link, origin xyz=-0.005 0.07 0 rpy=0 0 0, axis 0 0 1, limit lower=0 upper=0.79 effort=160.0 velocity=0.5
- added joint left_finger2_base_joint: type revolute, parent left_hand_link, child left_finger2_base_link, origin xyz=0 0.025 0 rpy=0 1.57 0, axis 0 0 1, limit lower=-3.14 upper=0 effort=160.0 velocity=0.5
- added joint left_finger2_joint1: type revolute, parent left_finger2_base_link, child left_finger2_1_link, origin xyz=-0.05 0 0.036 rpy=0 1.57 1.57, axis 0 0 1, limit lower=0 upper=2.44 effort=160.0 velocity=0.5
- added joint left_finger2_joint2: type revolute, parent left_finger2_1_link, child left_finger2_2_link, origin xyz=-0.005 0.07 0 rpy=0 0 0, axis 0 0 1, limit lower=0 upper=0.79 effort=160.0 velocity=0.5
- added joint left_finger3_joint1: type revolute, parent left_hand_link, child left_finger3_1_link, origin xyz=0.03 0 -0.05 rpy=1.57 3.14 0, axis 0 0 1, limit lower=0 upper=2.44 effort=160.0 velocity=0.5
- added joint left_finger3_joint2: type revolute, parent left_finger3_1_link, child left_finger3_2_link, origin xyz=-0.005 0.07 0 rpy=0 0 0, axis 0 0 1, limit lower=0 upper=0.79 effort=160.0 velocity=0.5
- added joint left_fixed_joint1: type fixed, parent left_arm7_link, child left_fts_link, origin xyz=0 0 0.065 rpy=-1.57 -1.57 0
- added joint left_fixed_joint2: type fixed, parent left_fts_link, child left_adapter_link, origin xyz=0.04 0 0 rpy=0 0 0
- added joint left_fixed_joint3: type fixed, parent left_adapter_link, child left_hand_link, origin xyz=0.06 0 0 rpy=0 0 0
- added joint left_fixed_joint4: type fixed, parent left_hand_link, child left_hand_sensor_link, origin xyz=0.035 0 0 rpy=0 0 0
- added joint left_fixed_joint5: type fixed, parent left_finger3_2_link, child left_finger3_tip_link, origin xyz=-0.028 0.022 0 rpy=0 0 1.97
- added joint left_fixed_joint6: type fixed, parent left_finger1_2_link, child left_finger1_tip_link, origin xyz=-0.028 0.022 0 rpy=0 0 1.97
- added joint left_fixed_joint7: type fixed, parent left_finger2_2_link, child left_finger2_tip_link, origin xyz=-0.028 0.022 0 rpy=0 0 1.97
- added joint left_joint0: type revolute, parent left_arm0_link, child left_arm1_link, origin xyz=0 0 0.2 rpy=0 0 0, axis 0 0 1, limit lower=-1.57 upper=2.62 effort=160.0 velocity=0.5
- added joint left_joint1: type revolute, parent left_arm1_link, child left_arm2_link, origin xyz=0 0 0.14 rpy=1.57 1.57 0, axis 0 0 1, limit lower=-1.66 upper=0.79 effort=160.0 velocity=0.5
- added joint left_joint2: type revolute, parent left_arm2_link, child left_arm3_link, origin xyz=-0.195 0 0 rpy=-1.57 0 1.57, axis 0 0 1, limit lower=-2.44 upper=1.57 effort=160.0 velocity=0.5
- added joint left_joint3: type revolute, parent left_arm3_link, child left_arm4_link, origin xyz=0 0 0.2 rpy=1.57 1.57 0, axis 0 0 1, limit lower=-2.88 upper=0.26 effort=160.0 velocity=0.5
- added joint left_joint4: type revolute, parent left_arm4_link, child left_arm5_link, origin xyz=-0.208 0 0 rpy=-1.57 0 1.57, axis 0 0 1, limit lower=-2.88 upper=2.88 effort=160.0 velocity=0.5
- added joint left_joint5: type revolute, parent left_arm5_link, child left_arm6_link, origin xyz=0 0 0.161 rpy=1.57 1.57 0, axis 0 0 1, limit lower=-2.09 upper=2.09 effort=160.0 velocity=0.5
- added joint left_joint6: type revolute, parent left_arm6_link, child left_arm7_link, origin xyz=-0.053 0 0 rpy=-1.57 0 1.57, axis 0 0 1, limit lower=-1.57 upper=2.88 effort=160.0 velocity=0.5
- added joint torso_to_left_joint0: type fixed, parent torso_link, child left_arm0_link, origin xyz=0 -0.045 0.297 rpy=1.57 -3.14 0

Commit message: first urdf complete

File: urdf/aros.urdf (robot description, URDF)
Before this commit: robot aros, 51 links, 50 joints
Links:
- link left_hand_sensor_link: geometry collision mesh filename=package://aros_description/meshes/hand/hand_sensor/link.dae; visual mesh filename=package://aros_description/meshes/hand/hand_sensor/body.dae
- link right_hand_sensor_link: geometry collision mesh filename=package://aros_description/meshes/hand/hand_sensor/link.dae; visual mesh filename=package://aros_description/meshes/hand/hand_sensor/body.dae
