Commit message: [-->] the first version of the description has been completed

File: urdf/common.xacro (robot description, xacro)
@@ -36,55 +36,161 @@
   <property name="vision_pitch" value="0.0" />
   <property name="vision_yaw" value="0.0" />
-  <!-- ********** Right arm link 0 ********** -->
-  <!-- Right arm link 0 Location: Add to the transform from torso to right arm 0-->
-  <property name="right_arm0_x" value="0.0" />
-  <property name="right_arm0_y" value="0.045" />
-  <property name="right_arm0_z" value="0.297" />
-  <property name="right_arm0_roll" value="-${M_PI/2}" />
-  <property name="right_arm0_pitch" value="-${M_PI}" />
-  <property name="right_arm0_yaw" value="0.0" />
-  <!-- ********** Right arm link 1 ********** -->
-  <!-- Right arm link 1 Location: Add to the transform from torso to right arm 1-->
-  <property name="right_arm1_x" value="0.0" />
-  <property name="right_arm1_y" value="0.0" />
-  <property name="right_arm1_z" value="0.2" />
-  <property name="right_arm1_roll" value="0.0" />
-  <property name="right_arm1_pitch" value="0.0" />
-  <property name="right_arm1_yaw" value="0.0" />
-  <!-- Right arm joint 1 limits-->
-  <property name="right_arm1_lower" value="-${153.0*M_PI/180.0}" />
-  <property name="right_arm1_upper" value="${M_PI/2}" />
-	  <!-- ********** Right arm link 1 ********** -->
-  <!-- Right arm link 1 Location: Add to the transform from torso to right arm 1-->
-  <property name="right_arm1_x" value="0.0" />
-  <property name="right_arm1_y" value="0.0" />
-  <property name="right_arm1_z" value="0.2" />
-  <property name="right_arm1_roll" value="0.0" />
-  <property name="right_arm1_pitch" value="0.0" />
-  <property name="right_arm1_yaw" value="0.0" />
-  <!-- Right arm joint 1 limits-->
-  <property name="right_arm1_lower" value="-${153.0*M_PI/180.0}" />
-  <property name="right_arm1_upper" value="${M_PI/2}" />
-  <!-- ********** Right arm link 2 ********** -->
-  <!-- Right arm link 2 Location: Add to the transform from torso to right arm 2-->
-  <property name="right_arm2_x" value="0.0" />
-  <property name="right_arm2_y" value="0.0" />
-  <property name="right_arm2_z" value="0.14" />
-  <property name="right_arm2_roll" value="${M_PI/2}" />
-  <property name="right_arm2_pitch" value="${M_PI/2}" />
-  <property name="right_arm2_yaw" value="0.0" />
-  <!-- Right arm joint 2 limits-->
-  <property name="right_arm2_lower" value="-${95*M_PI/180.0}" />
-  <property name="right_arm2_upper" value="${M_PI/4}" />
-  <!-- ********** Right arm link 3 ********** -->
-  <!-- Right arm link 3 Location: Add to the transform from torso to right arm 3-->
-  <property name="right_arm3_x" value="-0.195" />
-  <property name="right_arm3_y" value="0.0" />
-  <property name="right_arm3_z" value="0.0" />
-  <property name="right_arm3_roll" value="-${M_PI/2}" />
-  <property name="right_arm3_pitch" value="0.0" />
-  <property name="right_arm3_yaw" value="${M_PI/2}" />
-  <!-- Right arm joint 3 limits-->
-  <property name="right_arm3_lower" value="-${M_PI/2}" />
-  <property name="right_arm3_upper" value="${140*M_PI/180.0}" />
+  <!-- ********** arm link 0 ********** -->
+  <!-- arm link 0 Location: add to the transform from torso to right arm 0-->
+  <property name="arm0_x" value="0.0" />
+  <property name="arm0_y" value="0.045" />
+  <property name="arm0_z" value="0.297" />
+  <property name="arm0_roll" value="-${M_PI/2}" />
+  <property name="arm0_pitch" value="-${M_PI}" />
+  <property name="arm0_yaw" value="0.0" />
+  <!-- ********** arm link 1 ********** -->
+  <!-- arm link 1 Location: add to the transform from right arm 0 to right arm 1-->
+  <property name="arm1_x" value="0.0" />
+  <property name="arm1_y" value="0.0" />
+  <property name="arm1_z" value="0.2" />
+  <property name="arm1_roll" value="0.0" />
+  <property name="arm1_pitch" value="0.0" />
+  <property name="arm1_yaw" value="0.0" />
+  <!-- arm joint 1 limits : add the joint limits of the right arm link 1-->
+  <property name="arm1_lower" value="-${150.0*M_PI/180.0}" />
+  <property name="arm1_upper" value="${M_PI/2}" />
+  <!-- ********** arm link 2 ********** -->
+  <!-- arm link 2 Location: add to the transform from right arm 1 to right arm 2-->
+  <property name="arm2_x" value="0.0" />
+  <property name="arm2_y" value="0.0" />
+  <property name="arm2_z" value="0.14" />
+  <property name="arm2_roll" value="${M_PI/2}" />
+  <property name="arm2_pitch" value="${M_PI/2}" />
+  <property name="arm2_yaw" value="0.0" />
+  <!-- arm joint 2 limits : add the joint limits of the right arm link 2-->
+  <property name="arm2_lower" value="-${95*M_PI/180.0}" />
+  <property name="arm2_upper" value="${M_PI/4}" />
+  <!-- ********** arm link 3 ********** -->
+  <!-- arm link 3 Location: add to the transform from right arm 2 to right arm 3-->
+  <property name="arm3_x" value="-0.195" />
+  <property name="arm3_y" value="0.0" />
+  <property name="arm3_z" value="0.0" />
+  <property name="arm3_roll" value="-${M_PI/2}" />
+  <property name="arm3_pitch" value="0.0" />
+  <property name="arm3_yaw" value="${M_PI/2}" />
+  <!-- arm joint 3 limits : add the joint limits of the right arm link 3-->
+  <property name="arm3_lower" value="-${M_PI/2}" />
+  <property name="arm3_upper" value="${140*M_PI/180.0}" />
+  <!-- ********** arm link 4 ********** -->
+  <!-- arm link 4 Location: add to the transform from right arm 3 to right arm 4 -->
+  <property name="arm4_x" value="0.0" />
+  <property name="arm4_y" value="0.0" />
+  <property name="arm4_z" value="0.2" />
+  <property name="arm4_roll" value="${M_PI/2}" />
+  <property name="arm4_pitch" value="${M_PI/2}" />
+  <property name="arm4_yaw" value="0.0" />
+  <!-- arm joint 4 limits : add the joint limits of the right arm link 4 -->
+  <property name="arm4_lower" value="-${165*M_PI/180.0}" />
+  <property name="arm4_upper" value="${15*M_PI/180.0}" />
+  <!-- ********** arm link 5 ********** -->
+  <!-- arm link 5 Location: add to the transform from right arm 4 to right arm 5-->
+  <property name="arm5_x" value="-0.208" />
+  <property name="arm5_y" value="0.0" />
+  <property name="arm5_z" value="0.0" />
+  <property name="arm5_roll" value="-${M_PI/2}" />
+  <property name="arm5_pitch" value="0.0" />
+  <property name="arm5_yaw" value="${M_PI/2}" />
+  <!-- arm joint 5 limits : add the joint limits of the right arm link 5 -->
+  <property name="arm5_lower" value="-${165*M_PI/180.0}" />
+  <property name="arm5_upper" value="${165*M_PI/180.0}" />
+  <!-- ********** arm link 6 ********** -->
+  <!-- arm link 6 Location: add to the transform from right arm 5 to right arm 6-->
+  <property name="arm6_x" value="0.0" />
+  <property name="arm6_y" value="0.0" />
+  <property name="arm6_z" value="0.161" />
+  <property name="arm6_roll" value="${M_PI/2}" />
+  <property name="arm6_pitch" value="${M_PI/2}" />
+  <property name="arm6_yaw" value="0.0" />
+  <!-- arm joint 6 limits : add the joint limits of the right arm link 6 -->
+  <property name="arm6_lower" value="-${120*M_PI/180.0}" />
+  <property name="arm6_upper" value="${120*M_PI/180.0}" />
+  <!-- ********** arm link 7 ********** -->
+  <!-- arm link 7 Location: add to the transform from right arm 6 to right arm 7-->
+  <property name="arm7_x" value="-0.053" />
+  <property name="arm7_y" value="0.0" />
+  <property name="arm7_z" value="0.0" />
+  <property name="arm7_roll" value="-${M_PI/2}" />
+  <property name="arm7_pitch" value="0.0" />
+  <property name="arm7_yaw" value="${M_PI/2}" />
+  <!-- arm joint 7 limits : add the joint limits of the right arm link 7 -->
+  <property name="arm7_lower" value="-${M_PI/2}" />
+  <property name="arm7_upper" value="${165*M_PI/180.0}" />
+  <!-- ********** hand link fts ********** -->
+  <!-- hand link fts Location: add to the transform from right arm 7 to right hand fts -->
+  <property name="hand_fts_x" value="0.0" />
+  <property name="hand_fts_y" value="0.0" />
+  <property name="hand_fts_z" value="0.065" />
+  <property name="hand_fts_roll" value="-${M_PI/2}" />
+  <property name="hand_fts_pitch" value="-${M_PI/2}" />
+  <property name="hand_fts_yaw" value="0.0" />
+  <!-- ********** hand link adapter ********** -->
+  <!-- hand link adapter Location: add to the transform from right hand fts to right hand adapter -->
+  <property name="hand_adapter_x" value="0.04" />
+  <property name="hand_adapter_y" value="0.0" />
+  <property name="hand_adapter_z" value="0.0" />
+  <property name="hand_adapter_roll" value="0.0" />
+  <property name="hand_adapter_pitch" value="0.0" />
+  <property name="hand_adapter_yaw" value="0.0" />
+  <!-- ********** hand link barrett ********** -->
+  <!-- hand link barrett Location: add to the transform from right hand adapter to right hand barrett -->
+  <property name="hand_barrett_x" value="0.06" />
+  <property name="hand_barrett_y" value="0.0" />
+  <property name="hand_barrett_z" value="0.0" />
+  <property name="hand_barrett_roll" value="0.0" />
+  <property name="hand_barrett_pitch" value="0.0" />
+  <property name="hand_barrett_yaw" value="0.0" />
+  <!-- ********** hand link sensor ********** -->
+  <!-- hand link sensor Location: add to the transform from right hand barrett to right hand sensor -->
+  <property name="hand_sensor_x" value="0.035" />
+  <property name="hand_sensor_y" value="0.0" />
+  <property name="hand_sensor_z" value="0.0" />
+  <property name="hand_sensor_roll" value="0.0" />
+  <property name="hand_sensor_pitch" value="0.0" />
+  <property name="hand_sensor_yaw" value="0.0" />
+  <!-- ********** finger  base link ********** -->
+  <!-- finger base link Location: add to the transform from right hand barrett to right hand finger base -->
+  <property name="finger_base_x" value="0.0" />
+  <property name="finger_base_y" value="-0.025" />
+  <property name="finger_base_z" value="0.0" />
+  <property name="finger_base_roll" value="0.0" />
+  <property name="finger_base_pitch" value="${M_PI/2}" />
+  <property name="finger_base_yaw" value="0.0" />
+    <!-- finger base limits : add the joint limits of the right finger base -->
+  <property name="finger_base_lower" value="0.0" />
+  <property name="finger_base_upper" value="${M_PI}" />
+  <!-- ********** finger 1 link ********** -->
+  <!-- finger 1 link Location: add to the transform from right hand finger 1 base to right hand finger 1 -->
+  <property name="finger_1_x" value="-0.05" />
+  <property name="finger_1_y" value="0.0" />
+  <property name="finger_1_z" value="0.036" />
+  <property name="finger_1_roll" value="0.0" />
+  <property name="finger_1_pitch" value="${M_PI/2}" />
+  <property name="finger_1_yaw" value="${M_PI/2}" />
+    <!-- finger 1 limits : add the joint limits of the right finger 1 -->
+  <property name="finger_1_lower" value="0.0" />
+  <property name="finger_1_upper" value="${140*M_PI/180.0}" />
+  <!-- ********** finger 2 link ********** -->
+  <!-- finger 2 link Location: add to the transform from right hand finger 1 to right hand finger 2 -->
+  <property name="finger_2_x" value="-0.005" />
+  <property name="finger_2_y" value="0.07" />
+  <property name="finger_2_z" value="0.0" />
+  <property name="finger_2_roll" value="0.0" />
+  <property name="finger_2_pitch" value="0.0" />
+  <property name="finger_2_yaw" value="0.0" />
+    <!-- finger 2 limits : add the joint limits of the right finger 2 -->
+  <property name="finger_2_lower" value="0.0" />
+  <property name="finger_2_upper" value="${M_PI/4}" />
+  <!-- ********** finger tip link ********** -->
+  <!-- finger tip link Location: add to the transform from right hand finger 2 to right hand finger tip -->
+  <property name="finger_tip_x" value="-0.028" />
+  <property name="finger_tip_y" value="0.022" />
+  <property name="finger_tip_z" value="0.0" />
+  <property name="finger_tip_roll" value="0.0" />
+  <property name="finger_tip_pitch" value="0.0" />
+  <property name="finger_tip_yaw" value="${113*M_PI/180.0}" />
   </robot>

File: urdf/robot/aros.urdf.xacro (robot description, xacro)
@@ -9,4 +9,6 @@
 	<xacro:include filename="$(find aros_description)/urdf/fixed/fixed.urdf.xacro" />
 	<xacro:include filename="$(find aros_description)/urdf/arm/arm.urdf.xacro" />
+	<xacro:include filename="$(find aros_description)/urdf/hand/hand.urdf.xacro" />
+	<xacro:include filename="$(find aros_description)/urdf/hand/fingers.urdf.xacro" />
 	<xacro:aros_base_v0 name="base"/>
    <xacro:aros_fixed_v0 name="torso" parent="base">
@@ -22,16 +24,79 @@
     <origin xyz="${vision_x} ${vision_y} ${vision_z}" rpy="${vision_roll} ${vision_pitch} ${vision_yaw}" />
    </xacro:aros_fixed_v0>
-	<!-- Right arm-->
+	<!-- Right arm and hand -->
    <xacro:aros_arm_v0 prefix="right" name="arm0" parent="torso" link="0" revolute="false" lower="0" upper="0">
-    <origin xyz="${right_arm0_x} ${right_arm0_y} ${right_arm0_z}" rpy="${right_arm0_roll} ${right_arm0_pitch} ${right_arm0_yaw}" />
+    <origin xyz="${arm0_x} ${arm0_y} ${arm0_z}" rpy="${arm0_roll} ${arm0_pitch} ${arm0_yaw}" />
    </xacro:aros_arm_v0>
-   <xacro:aros_arm_v0 prefix="right" name="arm1" parent="arm0" link="1" revolute="true" lower="${right_arm1_lower}" upper="${right_arm1_upper}">
-    <origin xyz="${right_arm1_x} ${right_arm1_y} ${right_arm1_z}" rpy="${right_arm1_roll} ${right_arm1_pitch} ${right_arm1_yaw}" />
+   <xacro:aros_arm_v0 prefix="right" name="arm1" parent="arm0" link="1" revolute="true" lower="${arm1_lower}" upper="${arm1_upper}">
+    <origin xyz="${arm1_x} ${arm1_y} ${arm1_z}" rpy="${arm1_roll} ${arm1_pitch} ${arm1_yaw}" />
    </xacro:aros_arm_v0>
-   <xacro:aros_arm_v0 prefix="right" name="arm2" parent="arm1" link="2" revolute="true" lower="${right_arm2_lower}" upper="${right_arm2_upper}">
-    <origin xyz="${right_arm2_x} ${right_arm2_y} ${right_arm2_z}" rpy="${right_arm2_roll} ${right_arm2_pitch} ${right_arm2_yaw}" />
+   <xacro:aros_arm_v0 prefix="right" name="arm2" parent="arm1" link="2" revolute="true" lower="${arm2_lower}" upper="${arm2_upper}">
+    <origin xyz="${arm2_x} ${arm2_y} ${arm2_z}" rpy="${arm2_roll} ${arm2_pitch} ${arm2_yaw}" />
    </xacro:aros_arm_v0>
-   <xacro:aros_arm_v0 prefix="right" name="arm3" parent="arm2" link="3" revolute="true" lower="${right_arm3_lower}" upper="${right_arm3_upper}">
-    <origin xyz="${right_arm3_x} ${right_arm3_y} ${right_arm3_z}" rpy="${right_arm3_roll} ${right_arm3_pitch} ${right_arm3_yaw}" />
+   <xacro:aros_arm_v0 prefix="right" name="arm3" parent="arm2" link="3" revolute="true" lower="${arm3_lower}" upper="${arm3_upper}">
+    <origin xyz="${arm3_x} ${arm3_y} ${arm3_z}" rpy="${arm3_roll} ${arm3_pitch} ${arm3_yaw}" />
    </xacro:aros_arm_v0>
+   <xacro:aros_arm_v0 prefix="right" name="arm4" parent="arm3" link="4" revolute="true" lower="${arm4_lower}" upper="${arm4_upper}">
+    <origin xyz="${arm4_x} ${arm4_y} ${arm4_z}" rpy="${arm4_roll} ${arm4_pitch} ${arm4_yaw}" />
+   </xacro:aros_arm_v0>
+   <xacro:aros_arm_v0 prefix="right" name="arm5" parent="arm4" link="5" revolute="true" lower="${arm5_lower}" upper="${arm5_upper}">
+    <origin xyz="${arm5_x} ${arm5_y} ${arm5_z}" rpy="${arm5_roll} ${arm5_pitch} ${arm5_yaw}" />
+   </xacro:aros_arm_v0>
+   <xacro:aros_arm_v0 prefix="right" name="arm6" parent="arm5" link="6" revolute="true" lower="${arm6_lower}" upper="${arm6_upper}">
+    <origin xyz="${arm6_x} ${arm6_y} ${arm6_z}" rpy="${arm6_roll} ${arm6_pitch} ${arm6_yaw}" />
+   </xacro:aros_arm_v0>
+   <xacro:aros_arm_v0 prefix="right" name="arm7" parent="arm6" link="7" revolute="true" lower="${arm7_lower}" upper="${arm7_upper}">
+    <origin xyz="${arm7_x} ${arm7_y} ${arm7_z}" rpy="${arm7_roll} ${arm7_pitch} ${arm7_yaw}" />
+   </xacro:aros_arm_v0>
+   <xacro:aros_hand_v0 prefix="right" name="hand_fts" parent="arm7" collision="true">
+    <origin xyz="${hand_fts_x} ${hand_fts_y} ${hand_fts_z}" rpy="${hand_fts_roll} ${hand_fts_pitch} ${hand_fts_yaw}" />
+   </xacro:aros_hand_v0>
+   <xacro:aros_hand_v0 prefix="right" name="hand_adapter" parent="hand_fts" collision="false">
+    <origin xyz="${hand_adapter_x} ${hand_adapter_y} ${hand_adapter_z}" rpy="${hand_adapter_roll} ${hand_adapter_pitch} ${hand_adapter_yaw}" />
+   </xacro:aros_hand_v0>
+   <xacro:aros_hand_v0 prefix="right" name="hand_barrett" parent="hand_adapter" collision="true">
+    <origin xyz="${hand_barrett_x} ${hand_barrett_y} ${hand_barrett_z}" rpy="${hand_barrett_roll} ${hand_barrett_pitch} ${hand_barrett_yaw}" />
+   </xacro:aros_hand_v0>
+   <xacro:aros_hand_v0 prefix="right" name="hand_sensor" parent="hand_barrett" collision="true">
+    <origin xyz="${hand_sensor_x} ${hand_sensor_y} ${hand_sensor_z}" rpy="${hand_sensor_roll} ${hand_sensor_pitch} ${hand_sensor_yaw}" />
+   </xacro:aros_hand_v0>
+   <xacro:aros_fingers_v0 prefix="right" parent="hand_barrett" />
+	<!-- Left arm-->
+   <xacro:aros_arm_v0 prefix="left" name="arm0" parent="torso" link="0" revolute="false" lower="0" upper="0">
+    <origin xyz="${arm0_x} ${-arm0_y} ${arm0_z}" rpy="${-arm0_roll} ${arm0_pitch} ${arm0_yaw}" />
+   </xacro:aros_arm_v0>
+   <xacro:aros_arm_v0 prefix="left" name="arm1" parent="arm0" link="1" revolute="true" lower="${-arm1_upper}" upper="${-arm1_lower}">
+    <origin xyz="${arm1_x} ${arm1_y} ${arm1_z}" rpy="${arm1_roll} ${arm1_pitch} ${arm1_yaw}" />
+   </xacro:aros_arm_v0>
+   <xacro:aros_arm_v0 prefix="left" name="arm2" parent="arm1" link="2" revolute="true" lower="${arm2_lower}" upper="${arm2_upper}">
+    <origin xyz="${arm2_x} ${arm2_y} ${arm2_z}" rpy="${arm2_roll} ${arm2_pitch} ${arm2_yaw}" />
+   </xacro:aros_arm_v0>
+   <xacro:aros_arm_v0 prefix="left" name="arm3" parent="arm2" link="3" revolute="true" lower="${-arm3_upper}" upper="${-arm3_lower}">
+    <origin xyz="${arm3_x} ${arm3_y} ${arm3_z}" rpy="${arm3_roll} ${arm3_pitch} ${arm3_yaw}" />
+   </xacro:aros_arm_v0>
+   <xacro:aros_arm_v0 prefix="left" name="arm4" parent="arm3" link="4" revolute="true" lower="${arm4_lower}" upper="${arm4_upper}">
+    <origin xyz="${arm4_x} ${arm4_y} ${arm4_z}" rpy="${arm4_roll} ${arm4_pitch} ${arm4_yaw}" />
+   </xacro:aros_arm_v0>
+   <xacro:aros_arm_v0 prefix="left" name="arm5" parent="arm4" link="5" revolute="true" lower="${-arm5_upper}" upper="${-arm5_lower}">
+    <origin xyz="${arm5_x} ${arm5_y} ${arm5_z}" rpy="${arm5_roll} ${arm5_pitch} ${arm5_yaw}" />
+   </xacro:aros_arm_v0>
+   <xacro:aros_arm_v0 prefix="left" name="arm6" parent="arm5" link="6" revolute="true" lower="${arm6_lower}" upper="${arm6_upper}">
+    <origin xyz="${arm6_x} ${arm6_y} ${arm6_z}" rpy="${arm6_roll} ${arm6_pitch} ${arm6_yaw}" />
+   </xacro:aros_arm_v0>
+   <xacro:aros_arm_v0 prefix="left" name="arm7" parent="arm6" link="7" revolute="true" lower="${arm7_lower}" upper="${arm7_upper}">
+    <origin xyz="${arm7_x} ${arm7_y} ${arm7_z}" rpy="${arm7_roll} ${arm7_pitch} ${arm7_yaw}" />
+   </xacro:aros_arm_v0>
+   <xacro:aros_hand_v0 prefix="left" name="hand_fts" parent="arm7" collision="true">
+    <origin xyz="${hand_fts_x} ${hand_fts_y} ${hand_fts_z}" rpy="${hand_fts_roll} ${hand_fts_pitch} ${hand_fts_yaw}" />
+   </xacro:aros_hand_v0>
+   <xacro:aros_hand_v0 prefix="left" name="hand_adapter" parent="hand_fts" collision="false">
+    <origin xyz="${hand_adapter_x} ${hand_adapter_y} ${hand_adapter_z}" rpy="${hand_adapter_roll} ${hand_adapter_pitch} ${hand_adapter_yaw}" />
+   </xacro:aros_hand_v0>
+   <xacro:aros_hand_v0 prefix="left" name="hand_barrett" parent="hand_adapter" collision="true">
+    <origin xyz="${hand_barrett_x} ${hand_barrett_y} ${hand_barrett_z}" rpy="${hand_barrett_roll} ${hand_barrett_pitch} ${hand_barrett_yaw}" />
+   </xacro:aros_hand_v0>
+   <xacro:aros_hand_v0 prefix="left" name="hand_sensor" parent="hand_barrett" collision="true">
+    <origin xyz="${hand_sensor_x} ${hand_sensor_y} ${hand_sensor_z}" rpy="${hand_sensor_roll} ${hand_sensor_pitch} ${hand_sensor_yaw}" />
+   </xacro:aros_hand_v0>
+   <xacro:aros_fingers_v0 prefix="left" parent="hand_barrett" />
 </robot>
