Commit message: 

File: urdf/common.xacro (robot description, xacro)
@@ -139,26 +139,28 @@
   <!-- ********** hand link barrett ********** -->
   <!-- hand link barrett Location: add to the transform from right hand adapter to right hand barrett -->
-  <property name="hand_barrett_x" value="0.06" />
+  <property name="hand_barrett_x" value="0.088" />
   <property name="hand_barrett_y" value="0.0" />
   <property name="hand_barrett_z" value="0.0" />
-  <property name="hand_barrett_roll" value="0.0" />
+  <property name="hand_barrett_roll" value="${M_PI/2}" />
+  <!-- <property name="hand_barrett_roll" value="0.0" /> -->
   <property name="hand_barrett_pitch" value="0.0" />
-  <property name="hand_barrett_yaw" value="0.0" />
+  <property name="hand_barrett_yaw" value="${M_PI/2}" />
+  <!--<property name="hand_barrett_yaw" value="0.0" /> -->
   <!-- ********** hand link sensor ********** -->
   <!-- hand link sensor Location: add to the transform from right hand barrett to right hand sensor -->
-  <property name="hand_sensor_x" value="0.028" />
+  <property name="hand_sensor_x" value="0.0" />
   <property name="hand_sensor_y" value="0.0" />
   <property name="hand_sensor_z" value="0.0" />
-  <property name="hand_sensor_roll" value="${M_PI/2}" />
+  <property name="hand_sensor_roll" value="0.0" />
   <property name="hand_sensor_pitch" value="0.0" />
-  <property name="hand_sensor_yaw" value="${M_PI/2}" />
+  <property name="hand_sensor_yaw" value="0.0" />
   <!-- ********** finger  base link ********** -->
   <!-- finger base link Location: add to the transform from right hand barrett to right hand finger base -->
-  <property name="finger_base_x" value="0.0" />
-  <property name="finger_base_y" value="-0.025" />
-  <property name="finger_base_z" value="0.0" />
+  <property name="finger_base_x" value="-0.025" />
+  <property name="finger_base_y" value="0.0" />
+  <property name="finger_base_z" value="-0.028" />
   <property name="finger_base_roll" value="0.0" />
-  <property name="finger_base_pitch" value="${M_PI/2}" />
-  <property name="finger_base_yaw" value="0.0" />
+  <property name="finger_base_pitch" value="0.0" />
+  <property name="finger_base_yaw" value="${-M_PI/2}" />
     <!-- finger base limits : add the joint limits of the right finger base -->
   <property name="finger_base_lower" value="0.0" />

File: urdf/hand/fingers.urdf.xacro (robot description, xacro)
@@ -64,4 +64,5 @@
     <origin xyz="${finger_2_x} ${finger_2_y} ${finger_2_z}" rpy="${finger_2_roll} ${finger_2_pitch} ${finger_2_yaw}"/>
   </joint>
+<!--
 	<link name="${prefix}_finger1_tip_link">
 	 <visual>
@@ -76,4 +77,5 @@
     <origin xyz="${finger_tip_x} ${finger_tip_y} ${finger_tip_z}" rpy="${finger_tip_roll} ${finger_tip_pitch} ${finger_tip_yaw}"/>
   </joint>
+-->
 <!-- finger 2 -->
     <link name="${prefix}_finger2_base_link">
@@ -94,5 +96,5 @@
     <parent link="${prefix}_${parent}_link"/>
     <child link="${prefix}_finger2_base_link"/>
-    <origin xyz="${finger_base_x} ${-finger_base_y} ${finger_base_z}" rpy="${finger_base_roll} ${finger_base_pitch} ${finger_base_yaw}"/>
+    <origin xyz="${-finger_base_x} ${finger_base_y} ${finger_base_z}" rpy="${finger_base_roll} ${finger_base_pitch} ${finger_base_yaw}"/>
   </joint>
 	<link name="${prefix}_finger2_1_link">
@@ -134,4 +136,5 @@
     <origin xyz="${finger_2_x} ${finger_2_y} ${finger_2_z}" rpy="${finger_2_roll} ${finger_2_pitch} ${finger_2_yaw}"/>
   </joint>
+<!--
 	<link name="${prefix}_finger2_tip_link">
 	 <visual>
@@ -146,4 +149,5 @@
     <origin xyz="${finger_tip_x} ${finger_tip_y} ${finger_tip_z}" rpy="${finger_tip_roll} ${finger_tip_pitch} ${finger_tip_yaw}"/>
   </joint>
+-->
 <!-- finger 3 -->
 	<link name="${prefix}_finger3_1_link">
@@ -164,5 +168,5 @@
     <parent link="${prefix}_${parent}_link"/>
     <child link="${prefix}_finger3_1_link"/>
-    <origin xyz="${finger_1_z} ${finger_1_y} ${finger_1_x}" rpy="${finger_1_roll+M_PI/2} ${finger_1_pitch+M_PI/2} ${finger_1_yaw-M_PI/2}"/>
+    <origin xyz="${finger_1_y} ${finger_1_x} ${finger_1_z-0.028}" rpy="${finger_1_roll-M_PI/2} ${finger_1_pitch} ${finger_1_yaw}"/>
   </joint>
 	<link name="${prefix}_finger3_2_link">
@@ -185,4 +189,5 @@
     <origin xyz="${finger_2_x} ${finger_2_y} ${finger_2_z}" rpy="${finger_2_roll} ${finger_2_pitch} ${finger_2_yaw}"/>
   </joint>
+<!--
 	<link name="${prefix}_finger3_tip_link">
 	 <visual>
@@ -197,4 +202,5 @@
     <origin xyz="${finger_tip_x} ${finger_tip_y} ${finger_tip_z}" rpy="${finger_tip_roll} ${finger_tip_pitch} ${finger_tip_yaw}"/>
   </joint>
+-->
 </xacro:macro>
 </robot>

File: urdf/robot/aros.urdf.xacro (robot description, xacro)
@@ -49,4 +49,28 @@
     <origin xyz="${arm7_x} ${arm7_y} ${arm7_z}" rpy="${arm7_roll} ${arm7_pitch} ${arm7_yaw}" />
    </xacro:aros_arm_v0>
+	<!--
+   <xacro:aros_fixed_v0 name="right_arm7" parent="right_arm6">
+   <origin xyz="${arm7_x} ${arm7_y} ${arm7_z}" rpy="${arm7_roll} ${arm7_pitch} ${arm7_yaw}" />
+   </xacro:aros_fixed_v0>
+-->
+	<!--
+	<link name="right_arm7_link">
+	 <visual>
+        <geometry>
+              <mesh filename="package://aros_description/meshes/arm/link7/body.dae" />
+        </geometry>
+      </visual>
+	<collision>
+      <geometry>
+        <mesh filename="package://aros_description/meshes/arm/link7/link.dae" />
+      </geometry>
+    </collision>
+    </link>
+  <joint name="right_arm6_link_to_right_arm7_link" type="fixed">
+    <parent link="right_arm6_link"/>
+    <child link="right_arm7_link"/>
+    <origin xyz="${arm7_x} ${arm7_y} ${arm7_z}" rpy="${arm7_roll} ${arm7_pitch} ${arm7_yaw}" />
+  </joint>
+	-->
    <xacro:aros_hand_v0 prefix="right" name="hand_fts" parent="arm7" collision="true">
     <origin xyz="${hand_fts_x} ${hand_fts_y} ${hand_fts_z}" rpy="${hand_fts_roll} ${hand_fts_pitch} ${hand_fts_yaw}" />
@@ -58,8 +82,53 @@
     <origin xyz="${hand_barrett_x} ${hand_barrett_y} ${hand_barrett_z}" rpy="${hand_barrett_roll} ${hand_barrett_pitch} ${hand_barrett_yaw}" />
    </xacro:aros_hand_v0>
+	<!--
+	<xacro:aros_arm_v0 prefix="right" name="hand_barrett" parent="hand_adapter" link="7" revolute="true" lower="${arm7_lower}" upper="${arm7_upper}">
+    <origin xyz="${hand_barrett_x} ${hand_barrett_y} ${hand_barrett_z}" rpy="${hand_barrett_roll} ${hand_barrett_pitch} ${hand_barrett_yaw}" />
+   </xacro:aros_arm_v0>
+-->
+	<!--
+	 <link name="right_hand_barrett_link">
+	 <visual>
+        <geometry>
+              <mesh filename="package://aros_description/meshes/hand/hand_barrett/body.dae" />
+        </geometry>
+      </visual>
+	<collision>
+      <geometry>
+        <mesh filename="package://aros_description/meshes/hand/hand_barrett/link.dae" />
+      </geometry>
+    </collision>
+    </link>
+	 <joint name="right_joint7" type="revolute">
+		<axis xyz="0 0 1"/>
+		<limit effort="${EFFORT}" lower="${arm7_lower}" upper="${arm7_upper}" velocity="${VELOCITY}"/>
+		<parent link="right_hand_adapter_link"/>
+		<child link="right_hand_barrett_link"/>
+		<origin xyz="${hand_barrett_x} ${hand_barrett_y} ${hand_barrett_z}" rpy="${hand_barrett_roll} ${hand_barrett_pitch} ${hand_barrett_yaw}" />
+	  </joint>
+-->
    <xacro:aros_hand_v0 prefix="right" name="hand_sensor" parent="hand_barrett" collision="true">
     <origin xyz="${hand_sensor_x} ${hand_sensor_y} ${hand_sensor_z}" rpy="${hand_sensor_roll} ${hand_sensor_pitch} ${hand_sensor_yaw}" />
    </xacro:aros_hand_v0>
-   <xacro:aros_fingers_v0 prefix="right" parent="hand_barrett" />
+	<!--
+  <link name="right_hand_sensor_link">
+	 <visual>
+        <geometry>
+              <mesh filename="package://aros_description/meshes/hand/hand_sensor/body.dae" />
+        </geometry>
+      </visual>
+		<collision>
+		  <geometry>
+			<mesh filename="package://aros_description/meshes/hand/hand_sensor/link.dae" />
+		  </geometry>
+		</collision>
+    </link>
+  <joint name="right_endpoint" type="fixed">
+    <parent link="right_hand_barrett_link"/>
+    <child link="right_hand_sensor_link"/>
+    <origin xyz="${hand_sensor_x} ${hand_sensor_y} ${hand_sensor_z}" rpy="${hand_sensor_roll} ${hand_sensor_pitch} ${hand_sensor_yaw}" />
+  </joint>
+-->
+   <xacro:aros_fingers_v0 prefix="right" parent="hand_sensor" />
 	<!-- Left arm-->
    <xacro:aros_arm_v0 prefix="left" name="arm0" parent="torso" link="0" revolute="false" lower="0" upper="0">
@@ -99,4 +168,23 @@
     <origin xyz="${hand_sensor_x} ${hand_sensor_y} ${hand_sensor_z}" rpy="${hand_sensor_roll} ${hand_sensor_pitch} ${hand_sensor_yaw}" />
    </xacro:aros_hand_v0>
-   <xacro:aros_fingers_v0 prefix="left" parent="hand_barrett" />
+	<!--
+	  <link name="left_hand_sensor_link">
+	 <visual>
+        <geometry>
+              <mesh filename="package://aros_description/meshes/hand/hand_sensor/body.dae" />
+        </geometry>
+      </visual>
+		<collision>
+		  <geometry>
+			<mesh filename="package://aros_description/meshes/hand/hand_sensor/link.dae" />
+		  </geometry>
+		</collision>
+    </link>
+  <joint name="left_endpoint" type="fixed">
+    <parent link="left_hand_barrett_link"/>
+    <child link="left_hand_sensor_link"/>
+    <origin xyz="${hand_sensor_x} ${hand_sensor_y} ${hand_sensor_z}" rpy="${hand_sensor_roll} ${hand_sensor_pitch} ${hand_sensor_yaw}" />
+  </joint>
+-->
+   <xacro:aros_fingers_v0 prefix="left" parent="hand_sensor" />
 </robot>
