Commit message: 

File: urdf/base/base.urdf.xacro (robot description, xacro)
@@ -7,5 +7,5 @@
     <link name="${name}_link">
 	 <visual>
-        <!-- <origin xyz="0 0 0" rpy="0 0 0" /> -->
+        <origin xyz="0 0 0" rpy="0 0 0" />
         <geometry>
           <mesh filename="package://aros_description/meshes/base/body.dae" />
@@ -13,5 +13,5 @@
       </visual>
       <collision>
-        <!-- <origin xyz="0 0 0" rpy="0 0 0" /> -->
+        <origin xyz="0 0 0" rpy="0 0 0" />
         <geometry>
           <mesh filename="package://aros_description/meshes/base/link.dae" />
