Commit message: xacro right arm: almost completed

File: urdf/robot/aros.urdf.xacro (robot description, xacro)
@@ -5,5 +5,33 @@
        xmlns:xacro="http://playerstage.sourceforge.net/gazebo/xmlschema/#interface"
        name="aros" >
+	<xacro:include filename="$(find aros_description)/urdf/common.xacro" />
 	<xacro:include filename="$(find aros_description)/urdf/base/base.urdf.xacro" />
+	<xacro:include filename="$(find aros_description)/urdf/fixed/fixed.urdf.xacro" />
+	<xacro:include filename="$(find aros_description)/urdf/arm/arm.urdf.xacro" />
 	<xacro:aros_base_v0 name="base"/>
+   <xacro:aros_fixed_v0 name="torso" parent="base">
+    <origin xyz="${torso_x} ${torso_y} ${torso_z}" rpy="${torso_roll} ${torso_pitch} ${torso_yaw}" />
+   </xacro:aros_fixed_v0>
+   <xacro:aros_fixed_v0 name="pan_tilt" parent="torso">
+    <origin xyz="${pan_tilt_x} ${pan_tilt_y} ${pan_tilt_z}" rpy="${pan_tilt_roll} ${pan_tilt_pitch} ${pan_tilt_yaw}" />
+   </xacro:aros_fixed_v0>
+   <xacro:aros_fixed_v0 name="neck" parent="pan_tilt">
+    <origin xyz="${neck_x} ${neck_y} ${neck_z}" rpy="${neck_roll} ${neck_pitch} ${neck_yaw}" />
+   </xacro:aros_fixed_v0>
+   <xacro:aros_fixed_v0 name="vision" parent="neck">
+    <origin xyz="${vision_x} ${vision_y} ${vision_z}" rpy="${vision_roll} ${vision_pitch} ${vision_yaw}" />
+   </xacro:aros_fixed_v0>
+	<!-- Right arm-->
+   <xacro:aros_arm_v0 prefix="right" name="arm0" parent="torso" link="0" revolute="false" lower="0" upper="0">
+    <origin xyz="${right_arm0_x} ${right_arm0_y} ${right_arm0_z}" rpy="${right_arm0_roll} ${right_arm0_pitch} ${right_arm0_yaw}" />
+   </xacro:aros_arm_v0>
+   <xacro:aros_arm_v0 prefix="right" name="arm1" parent="arm0" link="1" revolute="true" lower="${right_arm1_lower}" upper="${right_arm1_upper}">
+    <origin xyz="${right_arm1_x} ${right_arm1_y} ${right_arm1_z}" rpy="${right_arm1_roll} ${right_arm1_pitch} ${right_arm1_yaw}" />
+   </xacro:aros_arm_v0>
+   <xacro:aros_arm_v0 prefix="right" name="arm2" parent="arm1" link="2" revolute="true" lower="${right_arm2_lower}" upper="${right_arm2_upper}">
+    <origin xyz="${right_arm2_x} ${right_arm2_y} ${right_arm2_z}" rpy="${right_arm2_roll} ${right_arm2_pitch} ${right_arm2_yaw}" />
+   </xacro:aros_arm_v0>
+   <xacro:aros_arm_v0 prefix="right" name="arm3" parent="arm2" link="3" revolute="true" lower="${right_arm3_lower}" upper="${right_arm3_upper}">
+    <origin xyz="${right_arm3_x} ${right_arm3_y} ${right_arm3_z}" rpy="${right_arm3_roll} ${right_arm3_pitch} ${right_arm3_yaw}" />
+   </xacro:aros_arm_v0>
 </robot>

Commit message: 

File: urdf/robot/aros.urdf.xacro (robot description, xacro)
@@ -49,28 +49,4 @@
     <origin xyz="${arm7_x} ${arm7_y} ${arm7_z}" rpy="${arm7_roll} ${arm7_pitch} ${arm7_yaw}" />
    </xacro:aros_arm_v0>
-	<!--
-   <xacro:aros_fixed_v0 name="right_arm7" parent="right_arm6">
-   <origin xyz="${arm7_x} ${arm7_y} ${arm7_z}" rpy="${arm7_roll} ${arm7_pitch} ${arm7_yaw}" />
-   </xacro:aros_fixed_v0>
--->
-	<!--
-	<link name="right_arm7_link">
-	 <visual>
-        <geometry>
-              <mesh filename="package://aros_description/meshes/arm/link7/body.dae" />
-        </geometry>
-      </visual>
-	<collision>
-      <geometry>
-        <mesh filename="package://aros_description/meshes/arm/link7/link.dae" />
-      </geometry>
-    </collision>
-    </link>
-  <joint name="right_arm6_link_to_right_arm7_link" type="fixed">
-    <parent link="right_arm6_link"/>
-    <child link="right_arm7_link"/>
-    <origin xyz="${arm7_x} ${arm7_y} ${arm7_z}" rpy="${arm7_roll} ${arm7_pitch} ${arm7_yaw}" />
-  </joint>
-	-->
    <xacro:aros_hand_v0 prefix="right" name="hand_fts" parent="arm7" collision="true">
     <origin xyz="${hand_fts_x} ${hand_fts_y} ${hand_fts_z}" rpy="${hand_fts_roll} ${hand_fts_pitch} ${hand_fts_yaw}" />
@@ -82,52 +58,7 @@
     <origin xyz="${hand_barrett_x} ${hand_barrett_y} ${hand_barrett_z}" rpy="${hand_barrett_roll} ${hand_barrett_pitch} ${hand_barrett_yaw}" />
    </xacro:aros_hand_v0>
-	<!--
-	<xacro:aros_arm_v0 prefix="right" name="hand_barrett" parent="hand_adapter" link="7" revolute="true" lower="${arm7_lower}" upper="${arm7_upper}">
-    <origin xyz="${hand_barrett_x} ${hand_barrett_y} ${hand_barrett_z}" rpy="${hand_barrett_roll} ${hand_barrett_pitch} ${hand_barrett_yaw}" />
-   </xacro:aros_arm_v0>
--->
-	<!--
-	 <link name="right_hand_barrett_link">
-	 <visual>
-        <geometry>
-              <mesh filename="package://aros_description/meshes/hand/hand_barrett/body.dae" />
-        </geometry>
-      </visual>
-	<collision>
-      <geometry>
-        <mesh filename="package://aros_description/meshes/hand/hand_barrett/link.dae" />
-      </geometry>
-    </collision>
-    </link>
-	 <joint name="right_joint7" type="revolute">
-		<axis xyz="0 0 1"/>
-		<limit effort="${EFFORT}" lower="${arm7_lower}" upper="${arm7_upper}" velocity="${VELOCITY}"/>
-		<parent link="right_hand_adapter_link"/>
-		<child link="right_hand_barrett_link"/>
-		<origin xyz="${hand_barrett_x} ${hand_barrett_y} ${hand_barrett_z}" rpy="${hand_barrett_roll} ${hand_barrett_pitch} ${hand_barrett_yaw}" />
-	  </joint>
--->
    <xacro:aros_hand_v0 prefix="right" name="hand_sensor" parent="hand_barrett" collision="true">
     <origin xyz="${hand_sensor_x} ${hand_sensor_y} ${hand_sensor_z}" rpy="${hand_sensor_roll} ${hand_sensor_pitch} ${hand_sensor_yaw}" />
    </xacro:aros_hand_v0>
-	<!--
-  <link name="right_hand_sensor_link">
-	 <visual>
-        <geometry>
-              <mesh filename="package://aros_description/meshes/hand/hand_sensor/body.dae" />
-        </geometry>
-      </visual>
-		<collision>
-		  <geometry>
-			<mesh filename="package://aros_description/meshes/hand/hand_sensor/link.dae" />
-		  </geometry>
-		</collision>
-    </link>
-  <joint name="right_endpoint" type="fixed">
-    <parent link="right_hand_barrett_link"/>
-    <child link="right_hand_sensor_link"/>
-    <origin xyz="${hand_sensor_x} ${hand_sensor_y} ${hand_sensor_z}" rpy="${hand_sensor_roll} ${hand_sensor_pitch} ${hand_sensor_yaw}" />
-  </joint>
--->
    <xacro:aros_fingers_v0 prefix="right" parent="hand_sensor" />
 	<!-- Left arm-->
@@ -168,23 +99,4 @@
     <origin xyz="${hand_sensor_x} ${hand_sensor_y} ${hand_sensor_z}" rpy="${hand_sensor_roll} ${hand_sensor_pitch} ${hand_sensor_yaw}" />
    </xacro:aros_hand_v0>
-	<!--
-	  <link name="left_hand_sensor_link">
-	 <visual>
-        <geometry>
-              <mesh filename="package://aros_description/meshes/hand/hand_sensor/body.dae" />
-        </geometry>
-      </visual>
-		<collision>
-		  <geometry>
-			<mesh filename="package://aros_description/meshes/hand/hand_sensor/link.dae" />
-		  </geometry>
-		</collision>
-    </link>
-  <joint name="left_endpoint" type="fixed">
-    <parent link="left_hand_barrett_link"/>
-    <child link="left_hand_sensor_link"/>
-    <origin xyz="${hand_sensor_x} ${hand_sensor_y} ${hand_sensor_z}" rpy="${hand_sensor_roll} ${hand_sensor_pitch} ${hand_sensor_yaw}" />
-  </joint>
--->
    <xacro:aros_fingers_v0 prefix="left" parent="hand_sensor" />
 </robot>
